File: Termostato-Diferencial-Mega.kicad_pcb (KiCad board)
At the start: 2 copper layers, 100 x 75 mm, 44 parts, among them J1 Screw_Terminal_01x15, P1 DISPLAYS_FILA1_ARRIBA, P2 DISPLAYS_FILA1_ABAJO, SW1 Coded_Switch, SW2 SW_PUSH, U1 74HC595, U2 74HC595, U3 74HC595

Commit message: color del pcb en 3d
Other:
- net class Default removed
- net class pista fina removed
